Commit message: modified my robot model

File: project2/src/my_robot/urdf/my_robot (original).xacro (robot description, xacro)
@@ -2,11 +2,11 @@
 <robot name="my_robot" xmlns:xacro="http://www.ros.org/wiki/xacro">
   <gazebo reference="left_wheel">
-      <material>Gazebo/Gray</material>
+      <material>Gazebo/Grey</material>
   </gazebo>
   <gazebo reference="right_wheel">
-      <material>Gazebo/Gray</material>
+      <material>Gazebo/Grey</material>
   </gazebo>
   <gazebo reference="camera">
-      <material>Gazebo/Black</material>
+      <material>Gazebo/Blue</material>
   </gazebo>
   <gazebo reference="chassis">
@@ -21,5 +21,5 @@
   </joint>
   <link name='chassis'>
-    <pose>0 0 0.1 0 0 0</pose>
+    <pose>0 0 0.2 0 0 0</pose>
     <inertial>
       <mass value="15.0"/>
@@ -31,8 +31,8 @@
       />
     </inertial>
-    <collision name='collision'>
+    <collision name='chassis_collision'>
       <origin xyz="0 0 0" rpy=" 0 0 0"/>
       <geometry>
-        <cylinder radius="0.25" length="0.15"/>
+        <cylinder radius=".25" length="0.2"/>
       </geometry>
     </collision>
@@ -40,5 +40,5 @@
       <origin xyz="0 0 0" rpy=" 0 0 0"/>
       <geometry>
-        <cylinder radius="0.25" length="0.15"/>
+        <cylinder radius=".4" length="0.2"/>
       </geometry>
     </visual>
@@ -46,5 +46,5 @@
       <origin xyz="-0.15 0 -0.05" rpy=" 0 0 0"/>
       <geometry>
-        <sphere radius="0.0999"/>
+        <sphere radius="0.1"/>
       </geometry>
     </collision>
@@ -58,5 +58,5 @@
       <origin xyz="0.15 0 -0.05" rpy=" 0 0 0"/>
       <geometry>
-        <sphere radius="0.0999"/>
+        <sphere radius="0.1"/>
       </geometry>
     </collision>
@@ -92,5 +92,5 @@
     </link>
     <joint type="continuous" name="left_wheel_hinge">
-      <origin xyz="0 0.175 0" rpy="0 0 0"/>
+      <origin xyz="0 0.2 0" rpy="0 0 0"/>
       <child link="left_wheel"/>
       <parent link="chassis"/>
@@ -123,5 +123,5 @@
     </link>
     <joint type="continuous" name="right_wheel_hinge">
-      <origin xyz="0 -0.175 0" rpy="0 0 0"/>
+      <origin xyz="0 -0.2 0" rpy="0 0 0"/>
       <child link="right_wheel"/>
       <parent link="chassis"/>
