Commit message: set my robot

File: project2/src/my_robot/urdf/my_robot.xacro (robot description, xacro)
@@ -2,14 +2,14 @@
 <robot name="my_robot" xmlns:xacro="http://www.ros.org/wiki/xacro">
   <gazebo reference="left_wheel">
-      <material>Gazebo/Gray</material>
+      <material>Gazebo/Grey</material>
   </gazebo>
   <gazebo reference="right_wheel">
-      <material>Gazebo/Gray</material>
+      <material>Gazebo/Grey</material>
   </gazebo>
   <gazebo reference="camera">
-      <material>Gazebo/Red</material>
+      <material>Gazebo/Blue</material>
   </gazebo>
   <gazebo reference="chassis">
-      <material>Gazebo/Blue</material>
+      <material>Gazebo/Orange</material>
   </gazebo>
   <xacro:include filename="$(find my_robot)/urdf/my_robot.gazebo"/>
@@ -21,5 +21,5 @@
   </joint>
   <link name='chassis'>
-    <pose>0 0 0.1 0 0 0</pose>
+    <pose>0 0 0.2 0 0 0</pose>
     <inertial>
       <mass value="15.0"/>
@@ -34,5 +34,5 @@
       <origin xyz="0 0 0" rpy=" 0 0 0"/>
       <geometry>
-        <box size=".4 .2 .1"/>
+        <cylinder radius=".25" length="0.2"/>
       </geometry>
     </collision>
@@ -40,5 +40,5 @@
       <origin xyz="0 0 0" rpy=" 0 0 0"/>
       <geometry>
-        <box size=".4 .2 .1"/>
+        <cylinder radius=".4" length="0.2"/>
       </geometry>
     </visual>
@@ -46,5 +46,5 @@
       <origin xyz="-0.15 0 -0.05" rpy=" 0 0 0"/>
       <geometry>
-        <sphere radius="0.0499"/>
+        <sphere radius="0.1"/>
       </geometry>
     </collision>
@@ -52,5 +52,5 @@
       <origin xyz="-0.15 0 -0.05" rpy=" 0 0 0"/>
       <geometry>
-        <sphere radius="0.05"/>
+        <sphere radius="0.1"/>
       </geometry>
     </visual>
@@ -58,5 +58,5 @@
       <origin xyz="0.15 0 -0.05" rpy=" 0 0 0"/>
       <geometry>
-        <sphere radius="0.0499"/>
+        <sphere radius="0.1"/>
       </geometry>
     </collision>
@@ -64,5 +64,5 @@
       <origin xyz="0.15 0 -0.05" rpy=" 0 0 0"/>
       <geometry>
-        <sphere radius="0.05"/>
+        <sphere radius="0.1"/>
       </geometry>
     </visual>
@@ -72,5 +72,5 @@
         <origin xyz="0 0 0" rpy=" 0 1.5707 1.5707"/>
         <geometry>
-          <cylinder radius="0.1" length="0.05"/>
+          <cylinder radius="0.15" length="0.05"/>
         </geometry>
       </collision>
@@ -78,5 +78,5 @@
         <origin xyz="0 0 0" rpy=" 0 1.5707 1.5707"/>
         <geometry>
-          <cylinder radius="0.1" length="0.05"/>
+          <cylinder radius="0.15" length="0.05"/>
         </geometry>
       </visual>
@@ -92,5 +92,5 @@
     </link>
     <joint type="continuous" name="left_wheel_hinge">
-      <origin xyz="0 0.15 0" rpy="0 0 0"/>
+      <origin xyz="0 0.2 0" rpy="0 0 0"/>
       <child link="left_wheel"/>
       <parent link="chassis"/>
@@ -103,5 +103,5 @@
         <origin xyz="0 0 0" rpy=" 0 1.5707 1.5707"/>
         <geometry>
-          <cylinder radius="0.1" length="0.05"/>
+          <cylinder radius="0.15" length="0.05"/>
         </geometry>
       </collision>
@@ -109,5 +109,5 @@
         <origin xyz="0 0 0" rpy=" 0 1.5707 1.5707"/>
         <geometry>
-          <cylinder radius="0.1" length="0.05"/>
+          <cylinder radius="0.15" length="0.05"/>
         </geometry>
       </visual>
@@ -123,5 +123,5 @@
     </link>
     <joint type="continuous" name="right_wheel_hinge">
-      <origin xyz="0 -0.15 0" rpy="0 0 0"/>
+      <origin xyz="0 -0.2 0" rpy="0 0 0"/>
       <child link="right_wheel"/>
       <parent link="chassis"/>
@@ -154,5 +154,5 @@
     </link>
     <joint type="fixed" name="camera_joint">
-      <origin xyz="0.2 0 0" rpy="0 0 0"/>
+      <origin xyz="0.25 0 0" rpy="0 0 0"/>
       <child link="camera"/>
       <parent link="chassis"/>

Commit message: Update my_robot.xacro
edit my robot model

File: project2/src/my_robot/urdf/my_robot.xacro (robot description, xacro)
@@ -1,17 +1,23 @@
 <?xml version='1.0'?>
 <robot name="my_robot" xmlns:xacro="http://www.ros.org/wiki/xacro">
-  <gazebo reference="left_wheel">
-      <material>Gazebo/Gray</material>
-  </gazebo>
-  <gazebo reference="right_wheel">
-      <material>Gazebo/Gray</material>
+<xacro:include filename="$(find my_robot)/urdf/my_robot.gazebo" />
+  <gazebo reference="chassis">
+    <material>Gazebo/White</material>
   </gazebo>
   <gazebo reference="camera">
-      <material>Gazebo/Black</material>
-  </gazebo>
-  <gazebo reference="chassis">
-      <material>Gazebo/White</material>
-  </gazebo>
-  <xacro:include filename="$(find my_robot)/urdf/my_robot.gazebo"/>
+    <material>Gazebo/Grey</material>
+  </gazebo>
+  <gazebo reference="left_front_wheel">
+    <material>Gazebo/Black</material>
+  </gazebo>
+  <gazebo reference="right_front_wheel">
+    <material>Gazebo/Black</material>
+  </gazebo>
+  <gazebo reference="left_rear_wheel">
+    <material>Gazebo/Black</material>
+  </gazebo>
+  <gazebo reference="right_rear_wheel">
+    <material>Gazebo/Black</material>
+  </gazebo>
   <link name="robot_footprint"></link>
   <joint name="robot_footprint_joint" type="fixed">
@@ -31,8 +37,8 @@
       />
     </inertial>
-    <collision name='collision'>
-      <origin xyz="0 0 0" rpy=" 0 0 0"/>
-      <geometry>
-        <cylinder radius="0.25" length="0.15"/>
+    <collision name='chassis_collision'>
+      <origin xyz="0 0 0" rpy=" 0 0 0"/>
+      <geometry>
+        <box size=".5 .2 .1"/>
       </geometry>
     </collision>
@@ -40,151 +46,201 @@
       <origin xyz="0 0 0" rpy=" 0 0 0"/>
       <geometry>
-        <cylinder radius="0.25" length="0.15"/>
-      </geometry>
-    </visual>
-    <collision name='back_caster_collision'>
-      <origin xyz="-0.15 0 -0.05" rpy=" 0 0 0"/>
-      <geometry>
-        <sphere radius="0.0999"/>
-      </geometry>
-    </collision>
-    <visual name='back_caster_visual'>
-      <origin xyz="-0.15 0 -0.05" rpy=" 0 0 0"/>
-      <geometry>
-        <sphere radius="0.1"/>
-      </geometry>
-    </visual>
-    <collision name='front_caster_collision'>
-      <origin xyz="0.15 0 -0.05" rpy=" 0 0 0"/>
-      <geometry>
-        <sphere radius="0.0999"/>
-      </geometry>
-    </collision>
-    <visual name='front_caster_visual'>
-      <origin xyz="0.15 0 -0.05" rpy=" 0 0 0"/>
-      <geometry>
-        <sphere radius="0.1"/>
-      </geometry>
-    </visual>
-  </link>
-    <link name='left_wheel'>
-      <collision name='left_wheel_collision'>
-        <origin xyz="0 0 0" rpy=" 0 1.5707 1.5707"/>
-        <geometry>
-          <cylinder radius="0.15" length="0.05"/>
-        </geometry>
-      </collision>
-      <visual name='left_wheel_visual'>
-        <origin xyz="0 0 0" rpy=" 0 1.5707 1.5707"/>
-        <geometry>
-          <cylinder radius="0.15" length="0.05"/>
-        </geometry>
-      </visual>
-      <inertial>
-        <mass value="5.0"/>
-        <origin xyz="0.0 0 0" rpy=" 0 0 0"/>
-        <inertia
-            ixx="0.1" ixy="0" ixz="0"
-            iyy="0.1" iyz="0"
-            izz="0.1"
-        />
-      </inertial>
-    </link>
-    <joint type="continuous" name="left_wheel_hinge">
-      <origin xyz="0 0.175 0" rpy="0 0 0"/>
-      <child link="left_wheel"/>
-      <parent link="chassis"/>
-      <axis xyz="0 1 0" rpy="0 0 0"/>
-      <limit effort="10000" velocity="1000"/>
-      <dynamics damping="1.0" friction="1.0"/>
-    </joint>
-    <link name='right_wheel'>
-      <collision name='right_wheel_collision'>
-        <origin xyz="0 0 0" rpy=" 0 1.5707 1.5707"/>
-        <geometry>
-          <cylinder radius="0.15" length="0.05"/>
-        </geometry>
-      </collision>
-      <visual name='right_wheel_visual'>
-        <origin xyz="0 0 0" rpy=" 0 1.5707 1.5707"/>
-        <geometry>
-          <cylinder radius="0.15" length="0.05"/>
-        </geometry>
-      </visual>
-      <inertial>
-        <mass value="5.0"/>
-        <origin xyz="0.0 0 0" rpy=" 0 0 0"/>
-        <inertia
-            ixx="0.1" ixy="0" ixz="0"
-            iyy="0.1" iyz="0"
-            izz="0.1"
-        />
-      </inertial>
-    </link>
-    <joint type="continuous" name="right_wheel_hinge">
-      <origin xyz="0 -0.175 0" rpy="0 0 0"/>
-      <child link="right_wheel"/>
-      <parent link="chassis"/>
-      <axis xyz="0 1 0" rpy="0 0 0"/>
-      <limit effort="10000" velocity="1000"/>
-      <dynamics damping="1.0" friction="1.0"/>
-    </joint>
-    <link name="camera">
-      <visual name='camera_visual'>
-        <origin xyz="0 0 0" rpy="0 0 0"/>
-        <geometry>
-          <box size="0.05 0.05 0.05"/>
-        </geometry>
-      </visual>
-      <collision name='camera_collision'>
-        <origin xyz="0 0 0" rpy="0 0 0"/>
-        <geometry>
-          <box size="0.05 0.05 0.05"/>
-        </geometry>
-      </collision>
-      <inertial>
-        <mass value="0.1"/>
-        <origin xyz="0.05 0.05 0.05" rpy=" 0 0 0"/>
-        <inertia
-            ixx="1e-6" ixy="0" ixz="0"
-            iyy="1e-6" iyz="0"
-            izz="1e-6"
-        />
-      </inertial>
-    </link>
-    <joint type="fixed" name="camera_joint">
-      <origin xyz="0.275 0 0" rpy="0 0 0"/>
-      <child link="camera"/>
-      <parent link="chassis"/>
-      <axis xyz="0 1 0" rpy="0 0 0"/>
-    </joint>
-    <link name="hokuyo">
-      <visual name='hokuyo_visual'>
-        <origin xyz="0 0 0" rpy="0 0 0"/>
-        <geometry>
-          <mesh filename="package://my_robot/meshes/hokuyo.dae"/>
-        </geometry>
-      </visual>
-      <collision name='hokuyo_collision'>
-        <origin xyz="0 0 0" rpy="0 0 0"/>
-        <geometry>
-          <box size="0.1 0.1 0.1"/>
-        </geometry>
-      </collision>
-      <inertial>
-        <mass value="1e-5"/>
-        <origin xyz="0.05 0.05 0.05" rpy=" 0 0 0"/>
-        <inertia
-            ixx="1e-6" ixy="0" ixz="0"
-            iyy="1e-6" iyz="0"
-            izz="1e-6"
-        />
-      </inertial>
-    </link>
-    <joint type="fixed" name="hokuyo_joint">
-      <origin xyz="0.15 0 0.1" rpy="0 0 0"/>
-      <child link="hokuyo"/>
-      <parent link="chassis"/>
-      <axis xyz="0 1 0" rpy="0 0 0"/>
-    </joint>
+        <box size=".5 .2 .1"/>
+      </geometry>
+    </visual>
+    <collision name='top_collision'>
+      <origin xyz=".175 0 .1" rpy=" 0 0 0"/>
+      <geometry>
+        <box size=".15 .2 .1"/>
+      </geometry>
+    </collision>
+    <visual name='top_visual'>
+      <origin xyz=".175 0 .1" rpy=" 0 0 0"/>
+      <geometry>
+        <box size=".15 .2 .1"/>
+      </geometry>
+    </visual>
+  </link>
+  <link name='left_front_wheel'>
+    <inertial>
+      <mass value="5.0"/>
+      <origin xyz="0.0 0 0" rpy=" 0 1.5707 1.5707"/>
+      <inertia
+          ixx="0.1" ixy="0" ixz="0"
+          iyy="0.1" iyz="0"
+          izz="0.1"
+      />
+    </inertial>
+    <collision name='left_front_wheel_collision'>
+      <origin xyz="0 0 0" rpy=" 0 1.5707 1.5707"/>
+      <geometry>
+        <cylinder length="0.02" radius="0.05"/>
+      </geometry>
+    </collision>
+    <visual name='left_front_wheel_visual'>
+      <origin xyz="0 0 0" rpy=" 0 1.5705 1.5707"/>
+      <geometry>
+        <cylinder length="0.02" radius="0.05"/>
+      </geometry>
+    </visual>
+  </link>
+  <joint type="continuous" name="left_front_wheel_hinge">
+    <origin xyz="0.15 0.1 -0.05" rpy="0 0 0"/>
+    <child link="left_front_wheel"/>
+    <parent link="chassis"/>
+    <axis xyz="0 1 0" rpy="0 0 0"/>
+    <limit effort="10000" velocity="1000"/>
+    <dynamics damping="1.0" friction="1.0"/>
+  </joint>
+  <link name='left_rear_wheel'>
+    <inertial>
+      <mass value="5.0"/>
+      <origin xyz="0.0 0 0" rpy=" 0 1.5707 1.5707"/>
+      <inertia
+          ixx="0.1" ixy="0" ixz="0"
+          iyy="0.1" iyz="0"
+          izz="0.1"
+      />
+    </inertial>
+    <collision name='left_rear_wheel_collision'>
+      <origin xyz="0 0 0" rpy=" 0 1.5707 1.5707"/>
+      <geometry>
+        <cylinder length="0.02" radius="0.05"/>
+      </geometry>
+    </collision>
+    <visual name='left_rear_wheel_visual'>
+      <origin xyz="0 0 0" rpy=" 0 1.5705 1.5707"/>
+      <geometry>
+        <cylinder length="0.02" radius="0.05"/>
+      </geometry>
+    </visual>
+  </link>
+  <joint type="continuous" name="left_rear_wheel_hinge">
+    <origin xyz="-0.15 0.1 -0.05" rpy="0 0 0"/>
+    <child link="left_rear_wheel"/>
+    <parent link="chassis"/>
+    <axis xyz="0 1 0" rpy="0 0 0"/>
+    <limit effort="10000" velocity="1000"/>
+    <dynamics damping="1.0" friction="1.0"/>
+  </joint>
+  <link name='right_front_wheel'>
+    <inertial>
+      <mass value="5.0"/>
+      <origin xyz="0.0 0 0" rpy=" 0 1.5707 1.5707"/>
+      <inertia
+          ixx="0.1" ixy="0" ixz="0"
+          iyy="0.1" iyz="0"
+          izz="0.1"
+      />
+    </inertial>
+    <collision name='right_front_wheel_collision'>
+      <origin xyz="0 0 0" rpy=" 0 1.5707 1.5707"/>
+      <geometry>
+        <cylinder length="0.02" radius="0.05"/>
+      </geometry>
+    </collision>
+    <visual name='right_front_wheel_visual'>
+      <origin xyz="0 0 0" rpy=" 0 1.5705 1.5707"/>
+      <geometry>
+        <cylinder length="0.02" radius="0.05"/>
+      </geometry>
+    </visual>
+  </link>
+  <joint type="continuous" name="right_front_wheel_hinge">
+    <origin xyz="0.15 -0.1 -0.05" rpy="0 0 0"/>
+    <child link="right_front_wheel"/>
+    <parent link="chassis"/>
+    <axis xyz="0 1 0" rpy="0 0 0"/>
+    <limit effort="10000" velocity="1000"/>
+    <dynamics damping="1.0" friction="1.0"/>
+  </joint>
+  <link name='right_rear_wheel'>
+    <inertial>
+      <mass value="5.0"/>
+      <origin xyz="0.0 0 0" rpy=" 0 1.5707 1.5707"/>
+      <inertia
+          ixx="0.1" ixy="0" ixz="0"
+          iyy="0.1" iyz="0"
+          izz="0.1"
+      />
+    </inertial>
+    <collision name='right_rear_wheel_collision'>
+      <origin xyz="0 0 0" rpy=" 0 1.5707 1.5707"/>
+      <geometry>
+        <cylinder length="0.02" radius="0.05"/>
+      </geometry>
+    </collision>
+    <visual name='right_rear_wheel_visual'>
+      <origin xyz="0 0 0" rpy=" 0 1.5705 1.5707"/>
+      <geometry>
+        <cylinder length="0.02" radius="0.05"/>
+      </geometry>
+    </visual>
+  </link>
+  <joint type="continuous" name="right_rear_wheel_hinge">
+    <origin xyz="-0.15 -0.1 -0.05" rpy="0 0 0"/>
+    <child link="right_rear_wheel"/>
+    <parent link="chassis"/>
+    <axis xyz="0 1 0" rpy="0 0 0"/>
+    <limit effort="10000" velocity="1000"/>
+    <dynamics damping="1.0" friction="1.0"/>
+  </joint>
+  <link name="camera">
+    <inertial>
+      <mass value="0.1"/>
+      <origin xyz="0 0 0" rpy=" 0 0 0"/>
+      <inertia
+          ixx="1e-6" ixy="0" ixz="0"
+          iyy="1e-6" iyz="0"
+          izz="1e-6"
+      />
+    </inertial>
+    <collision name='camera_collision'>
+      <origin xyz="0 0 0" rpy=" 0 0 0"/>
+      <geometry>
+        <box size="0.05 0.05 0.05"/>
+      </geometry>
+    </collision>
+    <visual name='camera_visual'>
+      <origin xyz="0 0 0" rpy=" 0 0 0"/>
+      <geometry>
+        <box size="0.05 0.05 0.05"/>
+      </geometry>
+    </visual>
+  </link>
+  <joint type="fixed" name="camera_joint">
+    <origin xyz="0.25 0 0" rpy="0 0 0"/>
+    <child link="camera"/>
+    <parent link="chassis"/>
+    <axis xyz="0 1 0" rpy="0 0 0"/>
+  </joint>
+  <link name="hokuyo">
+    <inertial>
+      <mass value="1e-5"/>
+      <origin xyz="0 0 0" rpy=" 0 0 0"/>
+      <inertia
+          ixx="1e-6" ixy="0" ixz="0"
+          iyy="1e-6" iyz="0"
+          izz="1e-6"
+      />
+    </inertial>
+    <collision name='hokuyo_collision'>
+      <origin xyz="0 0 0" rpy=" 0 0 0"/>
+      <geometry>
+        <box size="0.1 0.1 0.1"/>
+      </geometry>
+    </collision>
+    <visual name='hokuyo_visual'>
+      <origin xyz="0 0 0" rpy=" 0 0 0"/>
+      <geometry>
+        <mesh filename="package://my_robot/meshes/hokuyo.dae"/>
+      </geometry>
+    </visual>
+  </link>
+  <joint type="fixed" name="hokuyo_joint">
+    <origin xyz="0.175 0 0.175" rpy="0 0 0"/>
+    <child link="hokuyo"/>
+    <parent link="chassis"/>
+    <axis xyz="0 1 0" rpy="0 0 0"/>
+  </joint>
 </robot>

Commit message: Update my_robot.xacro

File: project2/src/my_robot/urdf/my_robot.xacro (robot description, xacro)
@@ -40,5 +40,5 @@
       <origin xyz="0 0 0" rpy=" 0 0 0"/>
       <geometry>
-        <box size=".5 .2 .1"/>
+        <box size=".5 .3 .1"/>
       </geometry>
     </collision>
@@ -46,5 +46,5 @@
       <origin xyz="0 0 0" rpy=" 0 0 0"/>
       <geometry>
-        <box size=".5 .2 .1"/>
+        <box size=".5 .3 .1"/>
       </geometry>
     </visual>
@@ -52,5 +52,5 @@
       <origin xyz=".175 0 .1" rpy=" 0 0 0"/>
       <geometry>
-        <box size=".15 .2 .1"/>
+        <box size=".15 .3 .1"/>
       </geometry>
     </collision>
@@ -58,5 +58,5 @@
       <origin xyz=".175 0 .1" rpy=" 0 0 0"/>
       <geometry>
-        <box size=".15 .2 .1"/>
+        <box size=".15 .3 .1"/>
       </geometry>
     </visual>
@@ -86,5 +86,5 @@
   </link>
   <joint type="continuous" name="left_front_wheel_hinge">
-    <origin xyz="0.15 0.1 -0.05" rpy="0 0 0"/>
+    <origin xyz="0.15 0.17 0" rpy="0 0 0"/>
     <child link="left_front_wheel"/>
     <parent link="chassis"/>
@@ -117,5 +117,5 @@
   </link>
   <joint type="continuous" name="left_rear_wheel_hinge">
-    <origin xyz="-0.15 0.1 -0.05" rpy="0 0 0"/>
+    <origin xyz="-0.15 0.17 0" rpy="0 0 0"/>
     <child link="left_rear_wheel"/>
     <parent link="chassis"/>
@@ -148,5 +148,5 @@
   </link>
   <joint type="continuous" name="right_front_wheel_hinge">
-    <origin xyz="0.15 -0.1 -0.05" rpy="0 0 0"/>
+    <origin xyz="0.15 -0.17 0" rpy="0 0 0"/>
     <child link="right_front_wheel"/>
     <parent link="chassis"/>
@@ -179,5 +179,5 @@
   </link>
   <joint type="continuous" name="right_rear_wheel_hinge">
-    <origin xyz="-0.15 -0.1 -0.05" rpy="0 0 0"/>
+    <origin xyz="-0.15 -0.17 0" rpy="0 0 0"/>
     <child link="right_rear_wheel"/>
     <parent link="chassis"/>
